File: air/PCB_gateway/untitled.sch (EAGLE design)
At the start: 16 parts, among them K1 351, Q1 S9013, U1 ESP32-DEVKITC-32D, U2 PC817X2NIP0F, X1 MSTBA2, X2 MSTBA2

Commit message: revisi PCB dan List komponen
Parts:
- removed S2: EG1224, EG1224:EG1224
Connections:
- net 3V3: no longer S2.3
- net GND: no longer S2.1, S2.SHIELD
- net M0: now also U1.IO15; no longer S2.2
Changed lines of the file:
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@@
 <part name="X1" library="con-phoenix-508" library_urn="urn:adsk.eagle:library:176" deviceset="MSTBA2" device="" package3d_urn="urn:adsk.eagle:package:9615/1"/>
 <part name="U$1" library="ethernet-mikroavr" deviceset="MINI_W5500" device=""/>
-<part name="S2" library="EG1224" deviceset="EG1224" device=""/>
 <part name="GND1" library="supply1" library_urn="urn:adsk.eagle:library:371" deviceset="GND" device=""/>
 <part name="D1" library="1N5819HW-7" deviceset="1N5819HW-7" device=""/>
@@
 <part name="GND2" library="supply1" library_urn="urn:adsk.eagle:library:371" deviceset="GND" device=""/>
 <part name="GND3" library="supply1" library_urn="urn:adsk.eagle:library:371" deviceset="GND" device=""/>
-<part name="GND5" library="supply1" library_urn="urn:adsk.eagle:library:371" deviceset="GND" device=""/>
 <part name="GND6" library="supply1" library_urn="urn:adsk.eagle:library:371" deviceset="GND" device=""/>
 <part name="P+3" library="supply1" library_urn="urn:adsk.eagle:library:371" deviceset="VCC" device=""/>
@@
 </instance>
 <instance part="U$1" gate="G$1" x="167.64" y="271.78" smashed="yes"/>
-<instance part="S2" gate="G$1" x="243.84" y="279.4" smashed="yes" rot="R270">
-<attribute name="NAME" x="252.73" y="284.48" size="1.27" layer="95" rot="R270"/>
-<attribute name="VALUE" x="234.95" y="284.48" size="1.27" layer="96" rot="R270" align="top-left"/>
-</instance>
 <instance part="GND1" gate="1" x="60.96" y="340.36" smashed="yes">
 <attribute name="VALUE" x="58.42" y="337.82" size="1.778" layer="96"/>
@@
 <instance part="GND3" gate="1" x="132.08" y="320.04" smashed="yes">
 <attribute name="VALUE" x="129.54" y="317.5" size="1.778" layer="96"/>
-</instance>
-<instance part="GND5" gate="1" x="248.92" y="259.08" smashed="yes">
-<attribute name="VALUE" x="246.38" y="256.54" size="1.778" layer="96"/>
 </instance>
 <instance part="GND6" gate="1" x="190.5" y="284.48" smashed="yes">
@@
 <wire x1="137.16" y1="322.58" x2="132.08" y2="322.58" width="0.1524" layer="91"/>
 <pinref part="GND3" gate="1" pin="GND"/>
-</segment>
-<segment>
-<pinref part="S2" gate="G$1" pin="SHIELD"/>
-<wire x1="238.76" y1="269.24" x2="238.76" y2="261.62" width="0.1524" layer="91"/>
-<pinref part="S2" gate="G$1" pin="1"/>
-<wire x1="238.76" y1="261.62" x2="248.92" y2="261.62" width="0.1524" layer="91"/>
-<wire x1="248.92" y1="261.62" x2="248.92" y2="269.24" width="0.1524" layer="91"/>
-<pinref part="GND5" gate="1" pin="GND"/>
-<junction x="248.92" y="261.62"/>
 </segment>
 <segment>
@@
 <label x="81.28" y="276.86" size="0.6096" layer="95" rot="R180" xref="yes"/>
 </segment>
-<segment>
-<pinref part="S2" gate="G$1" pin="3"/>
-<wire x1="243.84" y1="269.24" x2="243.84" y2="266.7" width="0.1524" layer="91"/>
-<label x="243.84" y="266.7" size="0.6096" layer="95" rot="R270" xref="yes"/>
-</segment>
 </net>
 <net name="M0" class="0">
@@
 </segment>
 <segment>
-<pinref part="S2" gate="G$1" pin="2"/>
-<wire x1="246.38" y1="289.56" x2="246.38" y2="292.1" width="0.1524" layer="91"/>
-<label x="246.38" y="292.1" size="0.6096" layer="95" rot="R90" xref="yes"/>
-</segment>
-</net>
+<pinref part="U1" gate="G$1" pin="IO15"/>
+<wire x1="124.46" y1="238.76" x2="127" y2="238.76" width="0.1524" layer="91"/>
+<label x="127" y="238.76" size="0.6096" layer="95" xref="yes"/>
+</segment>
+</net>

Commit message: revisi tanggal 24/02/2023
Parts:
- removed X2: MSTBA2, con-phoenix-508:MSTBA2
- added LED2, LED3: TLLY4400, led:TLLY4400
- added R4, R5: (no value), rcl:R-EU_R0805
- added X3: MSTBA3, con-phoenix-508:MSTBA3
Connections:
- new net LED_PRS: R4.2, U1.IO14
- new net LED_WRN: R5.2, U1.IO12
- new net N$11: LED3.A, R5.1
- new net N$9: LED2.A, R4.1
- net GND: now also LED2.C, LED3.C, X3-3.1
- net RXLORA_CONFIG: now also X3-2.1; no longer X2-2.1
- net TXLORA_CONFIG: now also X3-1.1; no longer X2-1.1
Changed lines of the file:
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@@
 <part name="P+4" library="supply1" library_urn="urn:adsk.eagle:library:371" deviceset="VCC" device=""/>
 <part name="GND7" library="supply1" library_urn="urn:adsk.eagle:library:371" deviceset="GND" device=""/>
-<part name="X2" library="con-phoenix-508" library_urn="urn:adsk.eagle:library:176" deviceset="MSTBA2" device="" package3d_urn="urn:adsk.eagle:package:9615/1"/>
 <part name="P+5" library="supply1" library_urn="urn:adsk.eagle:library:371" deviceset="VCC" device=""/>
 <part name="LED1" library="led" library_urn="urn:adsk.eagle:library:259" deviceset="TLLY4400" device="" package3d_urn="urn:adsk.eagle:package:15797/1"/>
@@
 <part name="GND8" library="supply1" library_urn="urn:adsk.eagle:library:371" deviceset="GND" device=""/>
 <part name="P+6" library="supply1" library_urn="urn:adsk.eagle:library:371" deviceset="VCC" device=""/>
+<part name="R4" library="rcl" library_urn="urn:adsk.eagle:library:334" deviceset="R-EU_" device="R0805" package3d_urn="urn:adsk.eagle:package:23553/2"/>
+<part name="LED2" library="led" library_urn="urn:adsk.eagle:library:259" deviceset="TLLY4400" device="" package3d_urn="urn:adsk.eagle:package:15797/1"/>
+<part name="R5" library="rcl" library_urn="urn:adsk.eagle:library:334" deviceset="R-EU_" device="R0805" package3d_urn="urn:adsk.eagle:package:23553/2"/>
+<part name="LED3" library="led" library_urn="urn:adsk.eagle:library:259" deviceset="TLLY4400" device="" package3d_urn="urn:adsk.eagle:package:15797/1"/>
+<part name="X3" library="con-phoenix-508" library_urn="urn:adsk.eagle:library:176" deviceset="MSTBA3" device="" package3d_urn="urn:adsk.eagle:package:9608/1"/>
+<part name="GND5" library="supply1" library_urn="urn:adsk.eagle:library:371" deviceset="GND" device=""/>
 </parts>
 <sheets>
@@
 <attribute name="VALUE" x="58.42" y="157.48" size="1.778" layer="96"/>
 </instance>
-<instance part="X2" gate="-1" x="165.1" y="233.68" smashed="yes">
-<attribute name="NAME" x="158.496" y="234.569" size="1.778" layer="95" rot="R180"/>
-</instance>
-<instance part="X2" gate="-2" x="165.1" y="228.6" smashed="yes">
-<attribute name="VALUE" x="157.48" y="224.79" size="1.778" layer="96"/>
-<attribute name="NAME" x="158.496" y="229.489" size="1.778" layer="95" rot="R180"/>
-</instance>
 <instance part="P+5" gate="VCC" x="182.88" y="284.48" smashed="yes">
 <attribute name="VALUE" x="180.34" y="281.94" size="1.778" layer="96" rot="R90"/>
@@
 <instance part="P+6" gate="VCC" x="200.66" y="251.46" smashed="yes">
 <attribute name="VALUE" x="198.12" y="248.92" size="1.778" layer="96" rot="R90"/>
+</instance>
+<instance part="R4" gate="G$1" x="215.9" y="241.3" smashed="yes" rot="R90">
+<attribute name="NAME" x="214.4014" y="237.49" size="1.778" layer="95" rot="R90"/>
+<attribute name="VALUE" x="219.202" y="237.49" size="1.778" layer="96" rot="R90"/>
+</instance>
+<instance part="LED2" gate="G$1" x="215.9" y="231.14" smashed="yes">
+<attribute name="NAME" x="219.456" y="226.568" size="1.778" layer="95" rot="R90"/>
+<attribute name="VALUE" x="221.615" y="226.568" size="1.778" layer="96" rot="R90"/>
+</instance>
+<instance part="R5" gate="G$1" x="226.06" y="241.3" smashed="yes" rot="R90">
+<attribute name="NAME" x="224.5614" y="237.49" size="1.778" layer="95" rot="R90"/>
+<attribute name="VALUE" x="229.362" y="237.49" size="1.778" layer="96" rot="R90"/>
+</instance>
+<instance part="LED3" gate="G$1" x="226.06" y="231.14" smashed="yes">
+<attribute name="NAME" x="229.616" y="226.568" size="1.778" layer="95" rot="R90"/>
+<attribute name="VALUE" x="231.775" y="226.568" size="1.778" layer="96" rot="R90"/>
+</instance>
+<instance part="X3" gate="-1" x="165.1" y="220.98" smashed="yes">
+<attribute name="NAME" x="158.496" y="221.869" size="1.778" layer="95" rot="R180"/>
+</instance>
+<instance part="X3" gate="-2" x="165.1" y="215.9" smashed="yes">
+<attribute name="NAME" x="158.496" y="216.789" size="1.778" layer="95" rot="R180"/>
+</instance>
+<instance part="X3" gate="-3" x="165.1" y="210.82" smashed="yes">
+<attribute name="VALUE" x="157.48" y="207.01" size="1.778" layer="96"/>
+<attribute name="NAME" x="158.496" y="211.709" size="1.778" layer="95" rot="R180"/>
+</instance>
+<instance part="GND5" gate="1" x="172.72" y="208.28" smashed="yes">
+<attribute name="VALUE" x="170.18" y="205.74" size="1.778" layer="96"/>
 </instance>
 </instances>
@@
 <pinref part="LED1" gate="G$1" pin="C"/>
 <wire x1="200.66" y1="223.52" x2="200.66" y2="226.06" width="0.1524" layer="91"/>
+<pinref part="LED2" gate="G$1" pin="C"/>
+<pinref part="LED3" gate="G$1" pin="C"/>
+<wire x1="215.9" y1="226.06" x2="226.06" y2="226.06" width="0.1524" layer="91"/>
+<wire x1="215.9" y1="226.06" x2="200.66" y2="226.06" width="0.1524" layer="91"/>
+<junction x="215.9" y="226.06"/>
+<junction x="200.66" y="226.06"/>
+</segment>
+<segment>
+<pinref part="X3" gate="-3" pin="1"/>
+<wire x1="170.18" y1="210.82" x2="172.72" y2="210.82" width="0.1524" layer="91"/>
+<pinref part="GND5" gate="1" pin="GND"/>
 </segment>
 </net>
@@
 <net name="TXLORA_CONFIG" class="0">
 <segment>
-<pinref part="X2" gate="-1" pin="1"/>
-<wire x1="170.18" y1="233.68" x2="175.26" y2="233.68" width="0.1524" layer="91"/>
-<label x="175.26" y="233.68" size="0.6096" layer="95" xref="yes"/>
-</segment>
-<segment>
 <pinref part="K1" gate="3" pin="S"/>
 <wire x1="78.74" y1="175.26" x2="78.74" y2="177.8" width="0.1524" layer="91"/>
@@
 <label x="93.98" y="177.8" size="0.6096" layer="95" xref="yes"/>
 </segment>
+<segment>
+<pinref part="X3" gate="-1" pin="1"/>
+<wire x1="170.18" y1="220.98" x2="172.72" y2="220.98" width="0.1524" layer="91"/>
+<label x="172.72" y="220.98" size="0.6096" layer="95" xref="yes"/>
+</segment>
 </net>
 <net name="RXLORA_CONFIG" class="0">
-<segment>
-<pinref part="X2" gate="-2" pin="1"/>
-<wire x1="170.18" y1="228.6" x2="175.26" y2="228.6" width="0.1524" layer="91"/>
-<label x="175.26" y="228.6" size="0.6096" layer="95" xref="yes"/>
-</segment>
 <segment>
 <pinref part="K1" gate="2" pin="S"/>
@@
 <label x="93.98" y="195.58" size="0.6096" layer="95" xref="yes"/>
 </segment>
+<segment>
+<pinref part="X3" gate="-2" pin="1"/>
+<wire x1="170.18" y1="215.9" x2="172.72" y2="215.9" width="0.1524" layer="91"/>
+<label x="172.72" y="215.9" size="0.6096" layer="95" xref="yes"/>
+</segment>
 </net>
 <net name="RXLORA_MICRO" class="0">
@@
 </segment>
 </net>
+<net name="N$9" class="0">
+<segment>
+<pinref part="R4" gate="G$1" pin="1"/>
+<pinref part="LED2" gate="G$1" pin="A"/>
+<wire x1="215.9" y1="236.22" x2="215.9" y2="233.68" width="0.1524" layer="91"/>
+</segment>
+</net>
+<net name="N$11" class="0">
+<segment>
+<pinref part="LED3" gate="G$1" pin="A"/>
+<pinref part="R5" gate="G$1" pin="1"/>
+<wire x1="226.06" y1="233.68" x2="226.06" y2="236.22" width="0.1524" layer="91"/>
+</segment>
+</net>
+<net name="LED_PRS" class="0">
+<segment>
+<pinref part="R4" gate="G$1" pin="2"/>
+<wire x1="215.9" y1="246.38" x2="215.9" y2="248.92" width="0.1524" layer="91"/>
+<label x="215.9" y="248.92" size="0.6096" layer="95" rot="R90" xref="yes"/>
+</segment>
+<segment>
+<pinref part="U1" gate="G$1" pin="IO14"/>
+<wire x1="83.82" y1="248.92" x2="81.28" y2="248.92" width="0.1524" layer="91"/>
+<label x="81.28" y="248.92" size="0.6096" layer="95" rot="R180" xref="yes"/>
+</segment>
+</net>
+<net name="LED_WRN" class="0">
+<segment>
+<pinref part="R5" gate="G$1" pin="2"/>
+<wire x1="226.06" y1="246.38" x2="226.06" y2="248.92" width="0.1524" layer="91"/>
+<label x="226.06" y="248.92" size="0.6096" layer="95" rot="R90" xref="yes"/>
+</segment>
+<segment>
+<pinref part="U1" gate="G$1" pin="IO12"/>
+<wire x1="83.82" y1="246.38" x2="81.28" y2="246.38" width="0.1524" layer="91"/>
+<label x="81.28" y="246.38" size="0.6096" layer="95" rot="R180" xref="yes"/>
+</segment>
+</net>
