File: air/PCB_node/untitled.sch (EAGLE design)
At the start: 32 parts, among them K1 351, K2 351, Q1 S9013, Q2 S9013, U1 ESP32-DEVKITC-32D, U2 PC817X2NIP0F, U3 PC817X2NIP0F, X1 MSTBA2, X2 MSTBA5, X3 MSTBA2, X4 MSTBA2, X5 MSTBA2

Commit message: revisi PCB dan List komponen
Parts:
- removed S2: EG1224, EG1224:EG1224
Connections:
- net 3V3: no longer S2.3
- net GND: no longer S2.1, S2.SHIELD
- net M0: now also U1.IO15; no longer S2.2
Changed lines of the file:
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@@
 <part name="MINI1" library="MINI560" deviceset="MINI560" device=""/>
 <part name="X1" library="con-phoenix-508" library_urn="urn:adsk.eagle:library:176" deviceset="MSTBA2" device="" package3d_urn="urn:adsk.eagle:package:9615/1"/>
-<part name="S2" library="EG1224" deviceset="EG1224" device=""/>
 <part name="GND1" library="supply1" library_urn="urn:adsk.eagle:library:371" deviceset="GND" device=""/>
 <part name="D1" library="1N5819HW-7" deviceset="1N5819HW-7" device=""/>
@@
 <part name="GND2" library="supply1" library_urn="urn:adsk.eagle:library:371" deviceset="GND" device=""/>
 <part name="GND3" library="supply1" library_urn="urn:adsk.eagle:library:371" deviceset="GND" device=""/>
-<part name="GND5" library="supply1" library_urn="urn:adsk.eagle:library:371" deviceset="GND" device=""/>
 <part name="X2" library="con-phoenix-508" library_urn="urn:adsk.eagle:library:176" deviceset="MSTBA5" device="" package3d_urn="urn:adsk.eagle:package:9612/1"/>
 <part name="ADS1" library="ds1115" deviceset="ADS1115" device=""/>
@@
 <attribute name="NAME" x="8.636" y="346.329" size="1.778" layer="95" rot="R180"/>
 </instance>
-<instance part="S2" gate="G$1" x="243.84" y="279.4" smashed="yes" rot="R270">
-<attribute name="NAME" x="252.73" y="284.48" size="1.27" layer="95" rot="R270"/>
-<attribute name="VALUE" x="234.95" y="284.48" size="1.27" layer="96" rot="R270" align="top-left"/>
-</instance>
 <instance part="GND1" gate="1" x="50.8" y="340.36" smashed="yes">
 <attribute name="VALUE" x="48.26" y="337.82" size="1.778" layer="96"/>
@@
 <instance part="GND3" gate="1" x="132.08" y="320.04" smashed="yes">
 <attribute name="VALUE" x="129.54" y="317.5" size="1.778" layer="96"/>
-</instance>
-<instance part="GND5" gate="1" x="248.92" y="259.08" smashed="yes">
-<attribute name="VALUE" x="246.38" y="256.54" size="1.778" layer="96"/>
 </instance>
 <instance part="X2" gate="-1" x="20.32" y="292.1" smashed="yes">
@@
 <wire x1="137.16" y1="322.58" x2="132.08" y2="322.58" width="0.1524" layer="91"/>
 <pinref part="GND3" gate="1" pin="GND"/>
-</segment>
-<segment>
-<pinref part="S2" gate="G$1" pin="SHIELD"/>
-<wire x1="238.76" y1="269.24" x2="238.76" y2="261.62" width="0.1524" layer="91"/>
-<pinref part="S2" gate="G$1" pin="1"/>
-<wire x1="238.76" y1="261.62" x2="248.92" y2="261.62" width="0.1524" layer="91"/>
-<wire x1="248.92" y1="261.62" x2="248.92" y2="269.24" width="0.1524" layer="91"/>
-<pinref part="GND5" gate="1" pin="GND"/>
-<junction x="248.92" y="261.62"/>
 </segment>
 <segment>
@@
 <junction x="78.74" y="274.32"/>
 </segment>
-<segment>
-<pinref part="S2" gate="G$1" pin="3"/>
-<wire x1="243.84" y1="269.24" x2="243.84" y2="266.7" width="0.1524" layer="91"/>
-<label x="243.84" y="266.7" size="0.6096" layer="95" rot="R270" xref="yes"/>
-</segment>
 </net>
 <net name="M0" class="0">
-<segment>
-<pinref part="S2" gate="G$1" pin="2"/>
-<wire x1="246.38" y1="289.56" x2="246.38" y2="292.1" width="0.1524" layer="91"/>
-<label x="246.38" y="292.1" size="0.6096" layer="95" rot="R90" xref="yes"/>
-</segment>
 <segment>
 <pinref part="EBYTEE220-900T22D1" gate="G$1" pin="M1"/>
@@
 <junction x="137.16" y="337.82"/>
 </segment>
-</net>
+<segment>
+<pinref part="U1" gate="G$1" pin="IO15"/>
+<wire x1="124.46" y1="238.76" x2="127" y2="238.76" width="0.1524" layer="91"/>
+<label x="127" y="238.76" size="0.6096" layer="95" xref="yes"/>
+</segment>
+</net>

Commit message: revisi tanggal 24/02/2023
Parts:
- removed LED1: TLLY4400, led:TLLY4400
- added D4: US1M-13, US1M-13:US1M-13
- added D5: SML-LXT0805IW-TR, SML-LXT0805IW-TR:SML-LXT0805IW-TR
- added K3: 351, relay:351
- added NEO-6MGPS1: (no value), NEO-6M GPS:NEO-6MGPS
- added Q3: S9013, S9013:S9013
- added R8, R9: (no value), rcl:R-EU_R0805
- added U4: PC817X2NIP0F, PC817X2NIP0F:PC817X2NIP0F
- added X6: MSTBA3, con-phoenix-508:MSTBA3
- X3: value MSTBA2 -> MSTBA4; device con-phoenix-508:MSTBA2 -> con-phoenix-508:MSTBA4
Connections:
- new net GND-VALVE: K32.S, X4-2.1
- new net N$11: Q3.B, U4.ET
- new net N$13: D4.A, K31.2, Q3.C
- new net N$4: R8.1, U4.A
- new net N$8: R9.2, U4.CT
- new net RX_GPS: NEO-6MGPS1.RX, U1.IO15
- new net TX_GPS: NEO-6MGPS1.TX, U1.IO14
- new net VALVE-POWER: R8.2, U1.IO13
- net GND: now also D5.C, K32.P, NEO-6MGPS1.GND, Q3.E, U4.C, X3-4.1, X6-3.1; no longer LED1.C, X4-2.1
- net M0: now also U1.IO4; no longer U1.IO15
- net N$1: now also D5.A; no longer LED1.A
- net RXLORA_CONFIG: now also X6-2.1; no longer X3-2.1
- net SCL: now also X3-3.1
- net SDA: now also X3-2.1
- net TXLORA_CONFIG: now also X6-1.1; no longer X3-1.1
- net VCC: now also D4.K, K31.1, NEO-6MGPS1.5V, R9.1, X3-1.1
Other:
- moved on the sheet: X3-1, X3-2, X5-1, X5-2
