File: air/PCB_node v1.1 with 2 lora/untitled.brd (EAGLE design)
At the start: 150 x 100 mm, 102 parts, among them J1 10118193-0001LF, J2 10118193-0001LF, K1 351, K2 351, K3 SRD-05VDC-SL-C, Q1 MMBT3904, Q2 MMBT3904, Q3 12MHz, Q4 S9013, Q5 S9013, Q6 S9013, Q7 12MHz, Q8 MMBT3904, Q9 MMBT3904, U1 CH340G, U10 ADS1115IDGSR, U2 ESP32-WROOM-32D, U3 AMS1117, U4 PC817X2NIP0F, U5 PC817X2NIP0F, U6 PC817X2NIP0F, U7 CH340G, U8 AMS1117, U9 ESP32-WROOM-32D, X1 MSTBA2, X2 MSTBA2, X3 MSTBA4, X4 MSTBA3, X5 MSTBA2, X6 MSTBA4, X7 C-GRID-02-70543

Commit message: PCB dasmeter dengan multidop
Parts:
- added D13, D14: US1M-13, US1M-13:DIOM5226X240N
- added EBYTEE220-900T22D2: (no value), EByte E220-900T22D:EBYTEE220-900T22D
- added JP1: (no value), adafruit:1X03
- added K4, K5: 351, relay:351
- added Q10, Q11: S9013, S9013:SOT95P240X120-3N
- added R22, R30: 1k, rcl:M0805
- added R29, R31: 10k, rcl:M0805
- added SJ1, SJ2, SJ3, SJ4: (no value), jumper:SJ
- added U11, U12: PC817X2NIP0F, PC817X2NIP0F:SOT254P975X400-4N
- added X8: MSTBA2, con-phoenix-508:MSTBA2
- moved C21 9.96 mm to (132.5, 49.0)
- moved U10 9.31 mm to (132.6, 45.0)
- moved ADS1 7.21 mm to (134.7, 46.1)
- moved NEO-6MGPS1 3.87 mm to (145.5, 12.9)
- moved R12 3.48 mm to (109.2, 11.3)
- moved R3 3.46 mm to (106.6, 11.5)
- moved D3 3.26 mm to (104.1, 11.5)
- moved SV1 1.38 mm to (41.4, 33.4)
- moved R11 1.26 mm to (107.3, 18.0)
- moved U5 0.67 mm to (96.6, 17.3)
- moved R9 0.30 mm to (83.3, 12.4)
Connections:
- new net M1: EBYTEE220-900T22D2.M0, EBYTEE220-900T22D2.M1, U9.29
- new net M2_CONFIGLORA: R30.2, U9.24
- new net M2_CONFIGRXLORA: JP1.2, K5.S2
- new net M2_CONFIGTXLORA: JP1.1, K5.S1
- new net M2_RX: K4.P2, U9.31
- new net M2_RXLORA: K5.O2, SJ4.2
- new net M2_RXLORA1: EBYTEE220-900T22D2.RXD, K5.P2
- new net M2_SWITCHGPS: R22.2, U9.11
- new net M2_TX: K4.P1, U9.30
- new net M2_TXLORA: K5.O1, SJ3.2
- new net M2_TXLORA1: EBYTEE220-900T22D2.TXD, K5.P1
- new net N$30: R22.1, U11.1
- new net N$31: Q10.1, U11.3
- new net N$32: R29.2, U11.4
- new net N$33: D13.A, K4.16, Q10.3
- new net N$34: R30.1, U12.1
- new net N$35: Q11.1, U12.3
- new net N$36: D14.A, K5.16, Q11.3
- new net N$38: R31.2, U12.4
- new net RX_LORA1: K4.S2, SJ2.1, SJ4.1
- new net TX_LORA1: K4.S1, SJ1.1, SJ3.1
- net CONFIG_LORA: now also U9.10; no longer U2.29
- net GND: now also EBYTEE220-900T22D2.GND, JP1.3, Q10.2, Q11.2, U11.2, U12.2
- net OUT+: now also D13.C, D14.C, EBYTEE220-900T22D2.VCC, K4.1, K5.1, R29.1, R31.1
- net RX_GPS: now also K4.O2; no longer U9.31
- net RX_LORA: now also SJ2.2
- net SCL1: now also X8.1
- net SDA1: now also X8.2
- net TX_GPS: now also K4.O1; no longer U9.30
- net TX_LORA: now also SJ1.2
Routing:
- net M1: track 0.00 -> 210.8 mm, vias 0 -> 2
- net M2_CONFIGLORA: track 0.00 -> 182.6 mm, vias 0 -> 4
- net SCL1: track 73.6 -> 249.7 mm, vias 1 -> 5
- net SDA1: track 68.0 -> 236.3 mm, vias 1 -> 5
- net CONFIG_LORA: track 51.6 -> 207.7 mm
- net TX_GPS: track 230.0 -> 102.5 mm, vias 1 -> 3
- net M2_SWITCHGPS: track 0.00 -> 127.1 mm, vias 0 -> 1
- net GND: track 970.0 -> 1082.7 mm, vias 5 -> 7
- net TX_LORA1: track 0.00 -> 109.3 mm, vias 0 -> 4
- net RX_GPS: track 0.00 -> 97.4 mm, vias 0 -> 2
- net RX_LORA1: track 0.00 -> 94.0 mm, vias 0 -> 3
- net OUT+: track 603.6 -> 689.7 mm, vias 4 -> 3
- net M2_TX: track 0.00 -> 83.6 mm, vias 0 -> 3
- net M2_CONFIGTXLORA: track 0.00 -> 77.6 mm
- net M2_RX: track 0.00 -> 75.1 mm, vias 0 -> 3
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Other:
- outline, holes or cut-outs redrawn
