File: air/PCB_node v1.1 with multidrop/untitled.brd (EAGLE design)
At the start: 150 x 100 mm, 113 parts, among them J1 10118193-0001LF, J2 10118193-0001LF, K1 351, K2 351, K3 SRD-05VDC-SL-C, K4 351, Q1 MMBT3904, Q10 S9013, Q2 MMBT3904, Q3 12MHz, Q4 S9013, Q5 S9013, Q6 S9013, Q7 12MHz, Q8 MMBT3904, Q9 MMBT3904, U1 CH340G, U10 ADS1115IDGSR, U11 PC817X2NIP0F, U2 ESP32-WROOM-32D, U3 AMS1117, U4 PC817X2NIP0F, U5 PC817X2NIP0F, U6 PC817X2NIP0F, U7 CH340G, U8 AMS1117, U9 ESP32-WROOM-32D, X1 MSTBA2, X2 MSTBA2, X3 MSTBA4, X4 MSTBA3, X5 MSTBA2, X6 MSTBA4, X7 C-GRID-02-70543, X8 MSTBA2

Commit message: desain PCB scada air
Parts:
- moved EBYTEE220-900T22D1 2.00 mm to (103.9, 63.4)
Routing:
- net GND: track 982.2 -> 987.5 mm
- net TX_LORA: track 140.4 -> 138.0 mm
- net RX_LORA: track 134.2 -> 132.2 mm
- net M1: track 73.3 -> 71.7 mm
- net OUT+: track 680.3 -> 681.2 mm
