File: air/PCB_scada air/untitled.sch (EAGLE design)
At the start: 55 parts, among them J1 10118193-0001LF, K1 351, Q1 MMBT3904, Q2 MMBT3904, Q3 12MHz, Q4 S9013, U1 CH340G, U2 ESP32-WROOM-32D, U3 AMS1117, U4 ADS1115IDGSR, U5 PC817X2NIP0F, X1 MSTBA2, X2 MSTBA3, X3 MSTBA4, X4 MSTBA5

Commit message: revisi scada air
Parts:
- removed R10: (no value), rcl:R-US_M0805
- removed X4: MSTBA5, con-phoenix-508:MSTBA5
- added X5: MSTBA4, con-phoenix-508:MSTBA4
Connections:
- removed net CYBLE5: R10.1, U2.IO33, X4-5.1
- net CYBLE1: now also X5-1.1; no longer X4-1.1
- net CYBLE2: now also X5-2.1; no longer X4-2.1
- net CYBLE3: now also X5-3.1; no longer X4-3.1
- net CYBLE4: now also X5-4.1; no longer X4-4.1
- net VCC: no longer R10.2
Changed lines of the file:
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@@
 <part name="R8" library="rcl" library_urn="urn:adsk.eagle:library:334" deviceset="R-US_" device="M0805" package3d_urn="urn:adsk.eagle:package:23556/2"/>
 <part name="R9" library="rcl" library_urn="urn:adsk.eagle:library:334" deviceset="R-US_" device="M0805" package3d_urn="urn:adsk.eagle:package:23556/2"/>
-<part name="R10" library="rcl" library_urn="urn:adsk.eagle:library:334" deviceset="R-US_" device="M0805" package3d_urn="urn:adsk.eagle:package:23556/2"/>
 <part name="P+5" library="supply1" library_urn="urn:adsk.eagle:library:371" deviceset="VCC" device=""/>
 <part name="R11" library="rcl" library_urn="urn:adsk.eagle:library:334" deviceset="R-EU_" device="0207/12" package3d_urn="urn:adsk.eagle:package:23489/1"/>
@@
 <part name="X3" library="con-phoenix-508" library_urn="urn:adsk.eagle:library:176" deviceset="MSTBA4" device="" package3d_urn="urn:adsk.eagle:package:9613/1"/>
 <part name="GND16" library="supply1" library_urn="urn:adsk.eagle:library:371" deviceset="GND" device=""/>
-<part name="X4" library="con-phoenix-508" library_urn="urn:adsk.eagle:library:176" deviceset="MSTBA5" device="" package3d_urn="urn:adsk.eagle:package:9612/1"/>
 <part name="D5" library="SML-LXT0805IW-TR" deviceset="SML-LXT0805IW-TR" device=""/>
 <part name="D6" library="SML-LXT0805IW-TR" deviceset="SML-LXT0805IW-TR" device=""/>
@@
 <part name="R16" library="rcl" library_urn="urn:adsk.eagle:library:334" deviceset="R-US_" device="M0805" package3d_urn="urn:adsk.eagle:package:23556/2" value="1k"/>
 <part name="P+6" library="supply1" library_urn="urn:adsk.eagle:library:371" deviceset="VCC" device=""/>
+<part name="X5" library="con-phoenix-508" library_urn="urn:adsk.eagle:library:176" deviceset="MSTBA4" device="" package3d_urn="urn:adsk.eagle:package:9613/1"/>
 </parts>
 <sheets>
@@
 <attribute name="VALUE" x="122.682" y="285.75" size="1.778" layer="96" rot="R90"/>
 </instance>
-<instance part="R10" gate="G$1" x="124.46" y="287.02" smashed="yes" rot="R90">
-<attribute name="NAME" x="122.9614" y="283.21" size="1.778" layer="95" rot="R90"/>
-<attribute name="VALUE" x="127.762" y="283.21" size="1.778" layer="96" rot="R90"/>
-</instance>
 <instance part="P+5" gate="VCC" x="124.46" y="304.8" smashed="yes">
 <attribute name="VALUE" x="121.92" y="302.26" size="1.778" layer="96" rot="R90"/>
@@
 <attribute name="VALUE" x="33.02" y="149.86" size="1.778" layer="96"/>
 </instance>
-<instance part="X4" gate="-1" x="78.74" y="195.58" smashed="yes">
-<attribute name="NAME" x="72.136" y="196.469" size="1.778" layer="95" rot="R180"/>
-</instance>
-<instance part="X4" gate="-2" x="78.74" y="190.5" smashed="yes">
-<attribute name="NAME" x="72.136" y="191.389" size="1.778" layer="95" rot="R180"/>
-</instance>
-<instance part="X4" gate="-3" x="78.74" y="185.42" smashed="yes">
-<attribute name="NAME" x="72.136" y="186.309" size="1.778" layer="95" rot="R180"/>
-</instance>
-<instance part="X4" gate="-4" x="78.74" y="180.34" smashed="yes">
-<attribute name="NAME" x="72.136" y="181.229" size="1.778" layer="95" rot="R180"/>
-</instance>
-<instance part="X4" gate="-5" x="78.74" y="175.26" smashed="yes">
-<attribute name="VALUE" x="71.12" y="171.45" size="1.778" layer="96"/>
-<attribute name="NAME" x="72.136" y="176.149" size="1.778" layer="95" rot="R180"/>
-</instance>
 <instance part="D5" gate="G$1" x="12.7" y="259.08" smashed="yes" rot="R90">
 <attribute name="NAME" x="8.62973125" y="257.04486875" size="1.780740625" layer="95" rot="R90"/>
@@
 <instance part="P+6" gate="VCC" x="17.78" y="287.02" smashed="yes">
 <attribute name="VALUE" x="15.24" y="284.48" size="1.778" layer="96" rot="R90"/>
+</instance>
+<instance part="X5" gate="-1" x="73.66" y="167.64" smashed="yes">
+<attribute name="NAME" x="67.056" y="168.529" size="1.778" layer="95" rot="R180"/>
+</instance>
+<instance part="X5" gate="-2" x="73.66" y="162.56" smashed="yes">
+<attribute name="NAME" x="67.056" y="163.449" size="1.778" layer="95" rot="R180"/>
+</instance>
+<instance part="X5" gate="-3" x="73.66" y="157.48" smashed="yes">
+<attribute name="NAME" x="67.056" y="158.369" size="1.778" layer="95" rot="R180"/>
+</instance>
+<instance part="X5" gate="-4" x="73.66" y="152.4" smashed="yes">
+<attribute name="VALUE" x="66.04" y="148.59" size="1.778" layer="96"/>
+<attribute name="NAME" x="67.056" y="153.289" size="1.778" layer="95" rot="R180"/>
 </instance>
 </instances>
@@
 <wire x1="119.38" y1="302.26" x2="119.38" y2="294.64" width="0.1524" layer="91"/>
 <junction x="114.3" y="302.26"/>
-<pinref part="R10" gate="G$1" pin="2"/>
 <wire x1="119.38" y1="302.26" x2="124.46" y2="302.26" width="0.1524" layer="91"/>
-<wire x1="124.46" y1="302.26" x2="124.46" y2="292.1" width="0.1524" layer="91"/>
 <junction x="119.38" y="302.26"/>
 <pinref part="P+5" gate="VCC" pin="VCC"/>
-<junction x="124.46" y="302.26"/>
 </segment>
 <segment>
@@
 </segment>
 <segment>
-<pinref part="X4" gate="-1" pin="1"/>
-<wire x1="83.82" y1="195.58" x2="86.36" y2="195.58" width="0.1524" layer="91"/>
-<label x="86.36" y="195.58" size="0.6096" layer="95" xref="yes"/>
+<pinref part="X5" gate="-1" pin="1"/>
+<wire x1="78.74" y1="167.64" x2="81.28" y2="167.64" width="0.1524" layer="91"/>
+<label x="81.28" y="167.64" size="0.6096" layer="95" xref="yes"/>
 </segment>
 </net>
@@
 </segment>
 <segment>
-<pinref part="X4" gate="-2" pin="1"/>
-<wire x1="83.82" y1="190.5" x2="86.36" y2="190.5" width="0.1524" layer="91"/>
-<label x="86.36" y="190.5" size="0.6096" layer="95" xref="yes"/>
+<pinref part="X5" gate="-2" pin="1"/>
+<wire x1="78.74" y1="162.56" x2="81.28" y2="162.56" width="0.1524" layer="91"/>
+<label x="81.28" y="162.56" size="0.6096" layer="95" xref="yes"/>
 </segment>
 </net>
@@
 </segment>
 <segment>
-<pinref part="X4" gate="-3" pin="1"/>
-<wire x1="83.82" y1="185.42" x2="86.36" y2="185.42" width="0.1524" layer="91"/>
-<label x="86.36" y="185.42" size="0.6096" layer="95" xref="yes"/>
+<pinref part="X5" gate="-3" pin="1"/>
+<wire x1="78.74" y1="157.48" x2="81.28" y2="157.48" width="0.1524" layer="91"/>
+<label x="81.28" y="157.48" size="0.6096" layer="95" xref="yes"/>
 </segment>
 </net>
@@
 </segment>
 <segment>
-<pinref part="X4" gate="-4" pin="1"/>
-<wire x1="83.82" y1="180.34" x2="86.36" y2="180.34" width="0.1524" layer="91"/>
-<label x="86.36" y="180.34" size="0.6096" layer="95" xref="yes"/>
-</segment>
-</net>
-<net name="CYBLE5" class="0">
-<segment>
-<pinref part="U2" gate="G$1" pin="IO33"/>
-<pinref part="R10" gate="G$1" pin="1"/>
-<wire x1="124.46" y1="281.94" x2="93.98" y2="281.94" width="0.1524" layer="91"/>
-<label x="124.46" y="281.94" size="0.6096" layer="95" xref="yes"/>
-</segment>
-<segment>
-<pinref part="X4" gate="-5" pin="1"/>
-<wire x1="83.82" y1="175.26" x2="86.36" y2="175.26" width="0.1524" layer="91"/>
-<label x="86.36" y="175.26" size="0.6096" layer="95" xref="yes"/>
-</segment>
-</net>
+<pinref part="X5" gate="-4" pin="1"/>
+<wire x1="78.74" y1="152.4" x2="81.28" y2="152.4" width="0.1524" layer="91"/>
+<label x="81.28" y="152.4" size="0.6096" layer="95" xref="yes"/>
+</segment>
+</net>
