File: air/gateway1/untitled.sch (EAGLE design)
At the start: 41 parts, among them J1 10118193-0001LF, K1 351, Q2 MMBT3904, Q3 MMBT3904, Q4 S9013, U1 CH340G, U2 ESP32-WROOM-32D, U3 AMS1117, U4 PC817X2NIP0F, X2 MSTBA3, X3 MSTBA3

Commit message: fix PCB
Connections:
- net M1: now also U2.IO25
Changed lines of the file:
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@@
 <label x="190.5" y="299.72" size="0.6096" layer="95" rot="R180" xref="yes"/>
+</segment>
+<segment>
+<pinref part="U2" gate="G$1" pin="IO25"/>
+<wire x1="71.12" y1="266.7" x2="73.66" y2="266.7" width="0.1524" layer="91"/>
+<label x="73.66" y="266.7" size="0.6096" layer="95" xref="yes"/>
 </segment>
 </net>
