File: air/PCB_gateway_scadaair/untitled.sch (EAGLE design)
At the start: 15 parts, among them K1 351, Q1 S9013, U1 ESP32-DEVKITC-32D, U2 PC817X2NIP0F, X1 MSTBA2, X3 MSTBA3

Commit message: revisi scada air
Parts:
- removed PS1: HLK-5M05, HLK-5M05:HLK-5M05
- removed X3: MSTBA3, con-phoenix-508:MSTBA3
- added D3, D4, D5: SS24, SS24:SS24
- added MINI1: (no value), MINI560:MINI560
- added PS2: HLK-20M12, HLK-20M12:HLK-20M12
- added X2: MSTBA2, con-phoenix-508:MSTBA2
- added X4, X5: C-GRID-02-70543, con-molex:C-GRID-02-70543
- D1: value 1N5819HW-7 -> SS24; device 1N5819HW-7:1N5819HW-7 -> SS24:SS24
Connections:
- removed net RXLORA_CONFIG: K12.S, X3-2.1
- removed net RXLORA_MICRO: K12.O, U1.IO17
- removed net TXLORA_CONFIG: K13.S, X3-1.1
- removed net TXLORA_MICRO: K13.O, U1.IO16
- new net 12V+: D1.K, D3.K, MINI1.IN+
- new net 5V+: D4.A, MINI1.OUT+, X4-2.S
- new net BATT+: D5.K, K12.P
- new net N$12: D5.A, X5-2.S
- new net N$5: D3.A, X2-1.1
- net GND: now also MINI1.IN-, MINI1.OUT-, PS2.-VO, X2-2.1, X4-1.S, X5-1.S; no longer PS1.-VO, X3-3.1
- net N$1: now also PS2.AC(L); no longer PS1.AC1
- net N$2: now also PS2.AC(N); no longer PS1.AC2
- net N$3: now also PS2.+VO; no longer PS1.+VO
- net RX_LORA: now also U1.IO17; no longer K12.P
- net TX_LORA: now also U1.IO16; no longer K13.P
- net VCC: now also D4.K, K12.S; no longer D1.K
